File: Hardware/Boards and Schematics/Traffic-tracker.brd (EAGLE design)
At the start: 70 x 70 mm, 6 parts, among them J2 POWER_JACKPTH

Commit message: Added protoboard section, cleaned up directory
Protoboard section with rails for 5V, 3v3, GND, and extra holes have
been added.

Trying to remove autosave .brd and .sch files
Parts:
- added JP1, JP3, JP4, JP5, JP6, JP7: (no value), SparkFun:1X06_HOLES_ONLY
Connections:
- new net VCC/2: JP3.1, JP3.2, JP3.3, JP3.4, JP3.5, JP3.6, WEMOS1.3V3
- net 5V: now also JP1.1, JP1.2, JP1.3, JP1.4, JP1.5, JP1.6
- net GND: now also JP4.1, JP4.2, JP4.3, JP4.4, JP4.5, JP4.6
Routing:
- net VCC/2: track 0.00 -> 91.6 mm
- net GND: track 0.00 -> 48.4 mm
- net 5V: track 124.7 -> 154.0 mm
Changed lines of the file:
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@@
 <setting verticaltext="up"/>
 </settings>
-<grid distance="0.05" unitdist="inch" unit="inch" style="lines" multiple="1" display="no" altdistance="0.025" altunitdist="inch" altunit="inch"/>
+<grid distance="0.1" unitdist="inch" unit="inch" style="lines" multiple="1" display="yes" altdistance="0.025" altunitdist="inch" altunit="inch"/>
 <layers>
 <layer number="1" name="Top" color="4" fill="1" visible="yes" active="yes"/>
@@
 <element name="V1" library="74ttl-din" package="DIL20" value="74245N" x="32.21" y="39.47"/>
 <element name="WEMOS1" library="esp8266modules" package="WEMOS-D1-MINI" value="" x="49.555" y="14.695" rot="R90"/>
+<element name="JP1" library="SparkFun" package="1X06_HOLES_ONLY" value="" x="5.08" y="20.32"/>
+<element name="JP3" library="SparkFun" package="1X06_HOLES_ONLY" value="" x="5.08" y="17.78"/>
+<element name="JP4" library="SparkFun" package="1X06_HOLES_ONLY" value="" x="5.08" y="15.24"/>
+<element name="JP5" library="SparkFun" package="1X06_HOLES_ONLY" value="" x="5.08" y="12.7"/>
+<element name="JP6" library="SparkFun" package="1X06_HOLES_ONLY" value="" x="5.08" y="10.16"/>
+<element name="JP7" library="SparkFun" package="1X06_HOLES_ONLY" value="" x="5.08" y="7.62"/>
 </elements>
 <signals>
@@
 <wire x1="54.61" y1="53.34" x2="65.55" y2="53.34" width="5.5" layer="1"/>
 <wire x1="65.55" y1="53.34" x2="65.55" y2="54.63" width="5.5" layer="1"/>
-<wire x1="59.715" y1="27.395" x2="59.715" y2="46.965" width="1.9304" layer="1"/>
-<wire x1="59.715" y1="46.965" x2="54.61" y2="52.07" width="1.9304" layer="1"/>
+<wire x1="59.715" y1="27.395" x2="59.715" y2="46.965" width="2.286" layer="1"/>
+<wire x1="59.715" y1="46.965" x2="54.61" y2="52.07" width="2.286" layer="1"/>
 <wire x1="54.61" y1="52.07" x2="54.61" y2="53.34" width="1.9304" layer="1"/>
 <wire x1="20.78" y1="35.66" x2="20.78" y2="43.28" width="1.27" layer="1"/>
@@
 <wire x1="59.715" y1="27.395" x2="59.715" y2="29.225" width="0.6096" layer="1"/>
 <wire x1="59.715" y1="29.225" x2="63.67" y2="33.18" width="0.6096" layer="1"/>
+<contactref element="JP1" pad="1"/>
+<contactref element="JP1" pad="2"/>
+<contactref element="JP1" pad="3"/>
+<contactref element="JP1" pad="4"/>
+<contactref element="JP1" pad="5"/>
+<contactref element="JP1" pad="6"/>
+<wire x1="20.78" y1="35.66" x2="20.78" y2="23.32" width="1.27" layer="1"/>
+<wire x1="20.78" y1="23.32" x2="17.78" y2="20.32" width="1.27" layer="1"/>
+<wire x1="17.78" y1="20.32" x2="15.24" y2="20.32" width="1.27" layer="1"/>
+<wire x1="15.24" y1="20.32" x2="12.7" y2="20.32" width="1.27" layer="1"/>
+<wire x1="12.7" y1="20.32" x2="10.16" y2="20.32" width="1.27" layer="1"/>
+<wire x1="10.16" y1="20.32" x2="7.62" y2="20.32" width="1.27" layer="1"/>
+<wire x1="7.62" y1="20.32" x2="5.08" y2="20.32" width="1.27" layer="1"/>
 </signal>
 <signal name="GND">
@@
 <vertex x="0" y="0"/>
 </polygon>
+<contactref element="JP4" pad="6"/>
+<contactref element="JP4" pad="5"/>
+<contactref element="JP4" pad="4"/>
+<contactref element="JP4" pad="3"/>
+<contactref element="JP4" pad="2"/>
+<contactref element="JP4" pad="1"/>
+<wire x1="17.78" y1="15.24" x2="20.32" y2="15.24" width="1.27" layer="16"/>
+<wire x1="20.32" y1="15.24" x2="37.465" y2="32.385" width="1.27" layer="16"/>
+<wire x1="37.465" y1="32.385" x2="42.545" y2="32.385" width="1.27" layer="16"/>
+<wire x1="42.545" y1="32.385" x2="43.815" y2="33.655" width="1.27" layer="16"/>
+<wire x1="43.815" y1="33.655" x2="43.815" y2="35.485" width="1.27" layer="16"/>
+<wire x1="43.815" y1="35.485" x2="43.64" y2="35.66" width="1.27" layer="16"/>
+<wire x1="17.78" y1="15.24" x2="15.24" y2="15.24" width="1.27" layer="16"/>
+<wire x1="15.24" y1="15.24" x2="12.7" y2="15.24" width="1.27" layer="16"/>
+<wire x1="12.7" y1="15.24" x2="10.16" y2="15.24" width="1.27" layer="16"/>
+<wire x1="10.16" y1="15.24" x2="7.62" y2="15.24" width="1.27" layer="16"/>
+<wire x1="7.62" y1="15.24" x2="5.08" y2="15.24" width="1.27" layer="16"/>
 </signal>
 <signal name="NEOPIX_DATA-IN_3V3">
@@
 <wire x1="26.035" y1="43.455" x2="25.86" y2="43.28" width="0.6096" layer="16"/>
 </signal>
+<signal name="VCC/2">
+<contactref element="WEMOS1" pad="3V3"/>
+<contactref element="JP3" pad="1"/>
+<contactref element="JP3" pad="2"/>
+<contactref element="JP3" pad="3"/>
+<contactref element="JP3" pad="4"/>
+<contactref element="JP3" pad="5"/>
+<contactref element="JP3" pad="6"/>
+<wire x1="59.715" y1="4.535" x2="59.715" y2="1.93" width="1.27" layer="1"/>
+<wire x1="59.715" y1="1.93" x2="59.055" y2="1.27" width="1.27" layer="1"/>
+<wire x1="59.055" y1="1.27" x2="3.175" y2="1.27" width="1.27" layer="1"/>
+<wire x1="3.175" y1="1.27" x2="1.905" y2="2.54" width="1.27" layer="1"/>
+<wire x1="1.905" y1="2.54" x2="1.905" y2="16.51" width="1.27" layer="1"/>
+<wire x1="1.905" y1="16.51" x2="3.175" y2="17.78" width="1.27" layer="1"/>
+<wire x1="3.175" y1="17.78" x2="5.08" y2="17.78" width="1.27" layer="1"/>
+<wire x1="5.08" y1="17.78" x2="7.62" y2="17.78" width="1.27" layer="1"/>
+<wire x1="7.62" y1="17.78" x2="10.16" y2="17.78" width="1.27" layer="1"/>
+<wire x1="10.16" y1="17.78" x2="12.7" y2="17.78" width="1.27" layer="1"/>
+<wire x1="12.7" y1="17.78" x2="15.24" y2="17.78" width="1.27" layer="1"/>
+<wire x1="15.24" y1="17.78" x2="17.78" y2="17.78" width="1.27" layer="1"/>
+</signal>
 </signals>
